File: MCT-1601.brd (EAGLE design)
At the start: 26.7 x 23.8 mm, 14 parts, among them J1 DUT, J2 Button, J3 D I/O, J5 A In, J6 Pwr, Q1 BC327

Commit message: Add files via upload
Parts:
- removed RLY1: W171-DIP-28, 00 Nik misc:DIL14-RELAY
- added D1: (no value), diode:D-2.5
- added K1: 351, relay:351
- moved Q1 1.27 mm to (3.81, 19.1)
Connections:
- new net N$1: J1.2, K1.P2
- new net N$4: J1.1, K1.P1
- net N$3: now also D1.A, K1.16; no longer RLY1.6
- net T1: now also K1.S1; no longer J1.1, RLY1.13, RLY1.14
- net T2: now also K1.S2; no longer J1.2, RLY1.1
- net T3: now also K1.O1, K1.O2; no longer RLY1.7, RLY1.8, RLY1.9
- net VCC: now also D1.C, K1.1; no longer RLY1.2
Routing:
- net T1: track 36.4 -> 16.8 mm
- net N$1: track 0.00 -> 19.4 mm
- net T3: track 49.3 -> 32.1 mm
- net N$4: track 0.00 -> 9.20 mm
- net N$3: track 18.8 -> 9.99 mm
- net VCC: track 4.34 -> 9.83 mm
- net GND: track 30.9 -> 36.0 mm
- net N$2: track 28.7 -> 32.0 mm
- net T2: track 26.9 -> 28.8 mm
Other:
- board text removed: "2"

Commit message: Add files via upload
Parts:
- added R8, R9: 10R, SparkFun-Resistors:AXIAL-0.1
- moved J2 4.58 mm to (24.1, 2.54), turned to 90 degrees
- moved D1 2.29 mm to (5.08, 15.2), turned to 90 degrees
- moved Q1 1.27 mm to (3.81, 20.3)
Connections:
- new net N$5: K1.O1, R8.P$2
- new net N$6: K1.O2, R9.P$2
- net T3: now also R8.P$1, R9.P$1; no longer K1.O1, K1.O2
Routing:
- net N$5: track 0.00 -> 20.5 mm
- net N$6: track 0.00 -> 15.3 mm
- net T2: track 28.8 -> 36.5 mm
- net N$2: track 32.0 -> 27.1 mm
- net N$1: track 19.4 -> 17.1 mm
- net N$3: track 9.99 -> 7.93 mm
- net GND: track 36.0 -> 34.8 mm, vias 0 -> 1
- net VCC: track 9.83 -> 9.20 mm
- net TEST_BUTTON: track 4.34 -> 3.81 mm

Commit message: Modified to support autodiagnostics on startup
Parts:
- removed R8, R9: 10R, SparkFun-Resistors:AXIAL-0.1
- moved D1 2.29 mm to (3.17, 14.0), turned to 180 degrees
- moved J2 1.91 mm to (24.1, 4.45)
- moved Q1 1.27 mm to (3.81, 19.1)
Connections:
- removed net N$5: K1.O1, R8.P$2
- removed net N$6: K1.O2, R9.P$2
- net T3: now also K1.O1, K1.O2; no longer R8.P$1, R9.P$1
Routing:
- net N$5: track 20.5 -> 0.00 mm
- net N$6: track 15.3 -> 0.00 mm
- net T2: track 36.5 -> 28.8 mm
- net N$1: track 17.1 -> 19.4 mm
- net N$3: track 7.93 -> 9.99 mm
- net N$2: track 27.1 -> 28.4 mm
- net TEST_BUTTON: track 3.81 -> 4.60 mm
- net VCC: track 9.20 -> 9.83 mm
- net GND: track 34.8 -> 35.0 mm, vias 1 -> 0

Commit message: Adding correct ec2 verion
Parts:
- moved R7 17.0 mm to (2.54, 12.7)
- moved D1 1.91 mm to (5.08, 14.0), turned to 90 degrees
- moved Q1 1.80 mm to (2.54, 20.3), turned to 270 degrees
- moved J2 1.42 mm to (24.8, 5.71), turned to 180 degrees
Connections:
- removed net N$1: J1.2, K1.P2
- removed net N$4: J1.1, K1.P1
- net T1: now also J1.1, K1.P1; no longer K1.S1
- net T2: now also J1.2, K1.P2; no longer K1.S2
Routing:
- net D7: track 2.54 -> 29.0 mm
- net N$2: track 28.4 -> 5.87 mm
- net N$1: track 19.4 -> 0.00 mm
- net T1: track 16.8 -> 29.6 mm
- net N$4: track 9.20 -> 0.00 mm
- net T2: track 28.8 -> 37.1 mm
- net GND: track 35.0 -> 40.4 mm
- net TEST_BUTTON: track 4.60 -> 7.62 mm
- net T3: track 32.1 -> 34.6 mm
- net N$3: track 9.99 -> 12.5 mm
Other:
- board text added: "Component Tester (C) Nik Berry 2016 ec 2"
- board text removed: "Component Tester (C) Nik Berry 2016 ec 1"

Commit message: Added diode value
Parts:
- D1: value (none) -> 1N4148
Changed lines of the file:
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@@
 <attribute name="VALUE" x="12.7" y="16.891" size="1.778" layer="27" ratio="10"/>
 </element>
-<element name="D1" library="diode" package="D-2.5" value="" x="5.08" y="13.97" smashed="yes" rot="R90">
-<attribute name="VALUE" x="7.493" y="12.319" size="1.27" layer="27" ratio="10" rot="R90"/>
+<element name="D1" library="diode" package="D-2.5" value="1N4148" x="5.08" y="13.97" smashed="yes" rot="R90">
+<attribute name="VALUE" x="4.318" y="12.319" size="0.6096" layer="27" ratio="10" rot="R90"/>
 </element>
 </elements>
